File: pcb/vmacpad-pcb/matrix.kicad_sch (KiCad schematic)
At the start: 0 parts

Commit message: Creating the PCB and additional parts
Parts:
- added D10, D12, D13, D14, D15, D17, D18, D2, D20, D22, D23, D25, D3, D5, D7, D8: SM4007, Diode_SMD:D_SOD-123F, symbol Diode:SM4007
- added K1, K10, K13, K14, K16, K17, K18, K2, K20, K4, K5, K6, K8, K9: 1u, acheron_MXH:MX100H, symbol Switch:SW_SPST
- added K12: 2.25u, acheron_MXH:MX225HR, symbol Switch:SW_SPST
Connections:
- new net: D23.2 (A), K18.2 (B)
- new net: D17.2 (A), K13.2 (B)
- new net: D20.2 (A), K16.2 (B)
- new net: D15.2 (A), K12.2 (B)
- new net: D22.2 (A), K17.2 (B)
- new net: D8.2 (A), K6.2 (B)
- new net: D2.2 (A), K1.2 (B)
- new net: D12.2 (A), K9.2 (B)
- new net: D10.2 (A), K8.2 (B)
- new net: D5.2 (A), K4.2 (B)
- new net: D25.2 (A), K20.2 (B)
- new net: D18.2 (A), K14.2 (B)
- new net: D13.2 (A), K10.2 (B)
- new net: D7.2 (A), K5.2 (B)
- new net: D3.2 (A), K2.2 (B)
- new net COL0: K1.1 (A), K2.1 (A), K4.1 (A)
- new net COL1: K5.1 (A), K6.1 (A), K8.1 (A)
- new net COL2: K10.1 (A), K12.1 (A), K9.1 (A)
- new net COL3: K13.1 (A), K14.1 (A), K16.1 (A)
- new net COL4: K17.1 (A), K18.1 (A), K20.1 (A)
- new net ENC_SW1: D14.2 (A)
- new net ROW0: D12.1 (K), D17.1 (K), D2.1 (K), D22.1 (K), D7.1 (K)
- new net ROW1: D13.1 (K), D18.1 (K), D23.1 (K), D3.1 (K), D8.1 (K)
- new net ROW2: D14.1 (K)
- new net ROW3: D10.1 (K), D15.1 (K), D20.1 (K), D25.1 (K), D5.1 (K)
Other:
- company: (none) -> 11kbd
- title: (none) -> VMacPad PCB - Switches

Commit message: Schematic Rev 1 done
Parts:
- D10, D12, D13, D14, D15, D17, D18, D2, D20, D22, D23, D25, D3, D5, D7, D8: footprint Diode_SMD:D_SOD-123F -> Diode_SMD:D_MELF

Commit message: Finalizing PCB
Parts:
- D1: renamed from D2; footprint Diode_SMD:D_MELF -> Diode_SMD:D_SOD-123F
- D10: renamed from D13; footprint Diode_SMD:D_MELF -> Diode_SMD:D_SOD-123F
- D11: renamed from D14; footprint Diode_SMD:D_MELF -> Diode_SMD:D_SOD-123F
- D12: renamed from D15; footprint Diode_SMD:D_MELF -> Diode_SMD:D_SOD-123F
- D13: renamed from D17; footprint Diode_SMD:D_MELF -> Diode_SMD:D_SOD-123F
- D14: renamed from D18; footprint Diode_SMD:D_MELF -> Diode_SMD:D_SOD-123F
- D16: renamed from D20; footprint Diode_SMD:D_MELF -> Diode_SMD:D_SOD-123F
- D17: renamed from D22; footprint Diode_SMD:D_MELF -> Diode_SMD:D_SOD-123F
- D18: renamed from D23; footprint Diode_SMD:D_MELF -> Diode_SMD:D_SOD-123F
- D2: renamed from D3; footprint Diode_SMD:D_MELF -> Diode_SMD:D_SOD-123F
- D20: renamed from D25; footprint Diode_SMD:D_MELF -> Diode_SMD:D_SOD-123F
- D4: renamed from D5; footprint Diode_SMD:D_MELF -> Diode_SMD:D_SOD-123F
- D5: renamed from D7; footprint Diode_SMD:D_MELF -> Diode_SMD:D_SOD-123F
- D6: renamed from D8; footprint Diode_SMD:D_MELF -> Diode_SMD:D_SOD-123F
- D8: renamed from D10; footprint Diode_SMD:D_MELF -> Diode_SMD:D_SOD-123F
- D9: renamed from D12; footprint Diode_SMD:D_MELF -> Diode_SMD:D_SOD-123F

Commit message: Fix properties
Parts:
- D1, D10, D11, D12, D13, D14, D16, D17, D18, D2, D20, D4, D5, D6, D8, D9: LCSC Part # C64898 -> (none); LCSC Part No (none) -> C64898; Package (none) -> SOD-123FL
- K1, K10, K12, K13, K14, K16, K17, K18, K2, K20, K4, K5, K6, K8, K9: LCSC Part # C5156480 -> (none); LCSC Part No (none) -> C5156480

Commit message: Fixes to part numbers and production
Parts:
- D1, D10, D11, D12, D13, D14, D16, D17, D18, D2, D20, D4, D5, D6, D8, D9: LCSC (none) -> C64898
- K1, K10, K12, K13, K14, K16, K17, K18, K2, K20, K4, K5, K6, K8, K9: LCSC (none) -> C5156480
