File: pcb/vmacpad-pcb/rgb.kicad_sch (KiCad schematic)
At the start: 1 part

Commit message: Creating the PCB and additional parts
Parts:
- added DL2, DL3, DL4, DL5, DL6: WS2812B, LED_SMD:LED_WS2812B_PLCC4_5.0x5.0mm_P3.2mm, symbol LED:WS2812B
- renumbered DL2 to DL1
Connections:
- net GND: now also DL2.3 (VSS), DL3.3 (VSS), DL4.3 (VSS), DL5.3 (VSS), DL6.3 (VSS)
- net VCC: now also DL2.1 (VDD), DL3.1 (VDD), DL4.1 (VDD), DL5.1 (VDD), DL6.1 (VDD)
- net at DL1.2 (DOUT): now also DL2.4 (DIN)
- new net: DL4.2 (DOUT), DL5.4 (DIN)
- new net: DL3.2 (DOUT), DL4.4 (DIN)
- new net: DL2.2 (DOUT), DL3.4 (DIN)
- new net: DL5.2 (DOUT), DL6.4 (DIN)
- no-connect marks 0 -> 1
Other:
- company: (none) -> 11kbd
- title: (none) -> VMacPad PCB - LEDs

Commit message: Fix properties
Parts:
- DL1, DL2, DL3, DL4, DL5, DL6: Package (none) -> SMD5050
Changed lines of the file:
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@@
+      (effects (font (size 1.27 1.27)) hide)
+    )
+    (property "Package" "SMD5050" (at 295.91 57.15 0)
       (effects (font (size 1.27 1.27)) hide)
     )
@@
       (effects (font (size 1.27 1.27)) hide)
     )
+    (property "Package" "SMD5050" (at 337.82 57.15 0)
+      (effects (font (size 1.27 1.27)) hide)
+    )
     (pin "1")
     (pin "2")
@@
       (effects (font (size 1.27 1.27)) hide)
     )
+    (property "Package" "SMD5050" (at 316.865 57.15 0)
+      (effects (font (size 1.27 1.27)) hide)
+    )
     (pin "1")
     (pin "2")
@@
       (effects (font (size 1.27 1.27)) hide)
     )
+    (property "Package" "SMD5050" (at 358.775 57.15 0)
+      (effects (font (size 1.27 1.27)) hide)
+    )
     (pin "1")
     (pin "2")
@@
       (effects (font (size 1.27 1.27)) hide)
     )
+    (property "Package" "SMD5050" (at 253.365 57.15 0)
+      (effects (font (size 1.27 1.27)) hide)
+    )
     (pin "1")
     (pin "2")
@@
       (effects (font (size 1.27 1.27)) hide)
     )
+    (property "Package" "SMD5050" (at 273.05 57.15 0)
+      (effects (font (size 1.27 1.27)) hide)
+    )

Commit message: Fixes to part numbers and production
Parts:
- DL1, DL2, DL3, DL4, DL5, DL6: LCSC (none) -> C2874885
Changed lines of the file:
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@@
+      (effects (font (size 1.27 1.27)) hide)
+    )
+    (property "LCSC" "C2874885" (at 295.91 57.15 0)
       (effects (font (size 1.27 1.27)) hide)
     )
@@
       (effects (font (size 1.27 1.27)) hide)
     )
+    (property "LCSC" "C2874885" (at 337.82 57.15 0)
+      (effects (font (size 1.27 1.27)) hide)
+    )
     (pin "1")
     (pin "2")
@@
       (effects (font (size 1.27 1.27)) hide)
     )
+    (property "LCSC" "C2874885" (at 316.865 57.15 0)
+      (effects (font (size 1.27 1.27)) hide)
+    )
     (pin "1")
     (pin "2")
@@
       (effects (font (size 1.27 1.27)) hide)
     )
+    (property "LCSC" "C2874885" (at 358.775 57.15 0)
+      (effects (font (size 1.27 1.27)) hide)
+    )
     (pin "1")
     (pin "2")
@@
       (effects (font (size 1.27 1.27)) hide)
     )
+    (property "LCSC" "C2874885" (at 253.365 57.15 0)
+      (effects (font (size 1.27 1.27)) hide)
+    )
     (pin "1")
     (pin "2")
@@
       (effects (font (size 1.27 1.27)) hide)
     )
+    (property "LCSC" "C2874885" (at 273.05 57.15 0)
+      (effects (font (size 1.27 1.27)) hide)
+    )
