File: pcb/vmacpad-pcb/vmacpad-pcb.kicad_pcb (KiCad board)
At the start: 2 copper layers, 156.1 x 117.1 mm, 30 parts, among them J1 TYPE-C-31-M12_13, SW1 SW_SPDT, U1 TPD4E05U06DQAR, U2 TXS0101DBVR, U3 STM32F401RCTx, Y1 16MHz

Commit message: Creating the PCB and additional parts
Parts:
- added D10: SM4007, Diode_SMD:D_SOD-123F, F.Cu at (165.3, 181.0)
- added D12: SM4007, Diode_SMD:D_SOD-123F, F.Cu at (170.8, 164.2)
- added D13: SM4007, Diode_SMD:D_SOD-123F, F.Cu at (170.8, 167.6)
- added D14: SM4007, Diode_SMD:D_SOD-123F, F.Cu at (170.8, 170.9)
- added D15: SM4007, Diode_SMD:D_SOD-123F, F.Cu at (170.8, 174.3)
- added D17: SM4007, Diode_SMD:D_SOD-123F, F.Cu at (170.8, 177.6)
- added D18: SM4007, Diode_SMD:D_SOD-123F, F.Cu at (170.8, 181.0)
- added D2: SM4007, Diode_SMD:D_SOD-123F, F.Cu at (165.3, 164.2)
- added D20: SM4007, Diode_SMD:D_SOD-123F, F.Cu at (176.3, 164.2)
- added D22: SM4007, Diode_SMD:D_SOD-123F, F.Cu at (176.3, 167.6)
- added D23: SM4007, Diode_SMD:D_SOD-123F, F.Cu at (176.3, 170.9)
- added D25: SM4007, Diode_SMD:D_SOD-123F, F.Cu at (176.3, 174.3)
- added D3: SM4007, Diode_SMD:D_SOD-123F, F.Cu at (165.3, 167.6)
- added D5: SM4007, Diode_SMD:D_SOD-123F, F.Cu at (165.3, 170.9)
- added D7: SM4007, Diode_SMD:D_SOD-123F, F.Cu at (165.3, 174.3)
- added D8: SM4007, Diode_SMD:D_SOD-123F, F.Cu at (165.3, 177.6)
- added DL1: WS2812B, LED_SMD:LED_WS2812B_PLCC4_5.0x5.0mm_P3.2mm, B.Cu at (211.9, 109.5)
- added DL3: WS2812B, LED_SMD:LED_WS2812B_PLCC4_5.0x5.0mm_P3.2mm, B.Cu at (211.9, 152.4)
- added DL4: WS2812B, LED_SMD:LED_WS2812B_PLCC4_5.0x5.0mm_P3.2mm, B.Cu at (211.9, 171.4)
- added DL5: WS2812B, LED_SMD:LED_WS2812B_PLCC4_5.0x5.0mm_P3.2mm, B.Cu at (161.9, 101.6)
- added DL6: WS2812B, LED_SMD:LED_WS2812B_PLCC4_5.0x5.0mm_P3.2mm, B.Cu at (123.8, 101.6)
- added J2: Conn_01x04_Pin, Connector_PinHeader_2.54mm:PinHeader_1x04_P2.54mm_Vertical, F.Cu at (109.6, 169.0)
- added K1: 1u, acheron_MXH:MX100H, F.Cu at (185.7, 109.5)
- added K10: 1u, acheron_MXH:MX100H, F.Cu at (142.9, 133.3)
- added K12: 2.25u, acheron_MXH:MX225HR, F.Cu at (159.5, 214.3)
- added K13: 1u, acheron_MXH:MX100H, F.Cu at (123.8, 114.3)
- added K14: 1u, acheron_MXH:MX100H, F.Cu at (123.8, 133.3)
- added K16: 1u, acheron_MXH:MX100H, F.Cu at (128.6, 214.3)
- added K17: 1u, acheron_MXH:MX100H, F.Cu at (100.0, 109.5)
- added K18: 1u, acheron_MXH:MX100H, F.Cu at (104.8, 133.3)
- added K2: 1u, acheron_MXH:MX100H, F.Cu at (181.0, 133.3)
- added K20: 1u, acheron_MXH:MX100H, F.Cu at (104.8, 214.3)
- added K4: 1u, acheron_MXH:MX100H, F.Cu at (214.3, 214.3)
- added K5: 1u, acheron_MXH:MX100H, F.Cu at (161.9, 114.3)
- added K6: 1u, acheron_MXH:MX100H, F.Cu at (161.9, 133.3)
- added K8: 1u, acheron_MXH:MX100H, F.Cu at (190.5, 214.3)
- added K9: 1u, acheron_MXH:MX100H, F.Cu at (142.9, 114.3)
- added SW2: Alps EM11, Rotary_Encoder:RotaryEncoder_Alps_EC11E-Switch_Vertical_H20mm, B.Cu at (148.2, 170.2)
- added SW3: BournsEM14, max_customs:BournsEM14, B.Cu at (142.9, 173.8)
- added U4: AMS1117-3.3, Package_TO_SOT_SMD:SOT-223-3_TabPin2, F.Cu at (116.9, 180.8)
- C1, C10, C2: footprint Capacitor_SMD:C_0805_2012Metric -> Capacitor_SMD:C_1206_3216Metric
- DL2: moved to B.Cu
- moved DL2 182.2 mm to (211.9, 133.3), turned to 180 degrees
- moved U2 162.9 mm to (101.0, 184.4)
- moved R1 154.3 mm to (109.5, 180.4)
- moved R2 154.3 mm to (109.5, 183.3)
- moved R3 154.3 mm to (109.5, 186.3)
- moved U1 153.3 mm to (123.5, 183.2)
- moved L1 152.3 mm to (124.7, 186.9)
- moved F1 148.6 mm to (114.7, 186.6)
- moved D1 147.7 mm to (101.5, 188.4)
- moved C2 146.7 mm to (114.8, 171.7)
- moved J1 142.7 mm to (123.1, 167.4)
- moved C1 142.1 mm to (114.8, 168.3)
- moved U3 140.0 mm to (121.8, 158.1)
- moved C3 125.5 mm to (112.4, 152.4)
- moved C4 125.5 mm to (112.4, 155.4)
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Connections:
- DL2 pad 2: unconnected-(DL2-DOUT-Pad2) -> Net-(DL2-DOUT)
- DL2 pad 4: RGB_5V -> Net-(DL1-DOUT)
- U3 pad 20: unconnected-(U3-PA4-Pad20) -> COL0
- U3 pad 21: unconnected-(U3-PA5-Pad21) -> COL1
- U3 pad 22: unconnected-(U3-PA6-Pad22) -> COL2
- U3 pad 23: unconnected-(U3-PA7-Pad23) -> COL3
- U3 pad 24: unconnected-(U3-PC4-Pad24) -> ENC_PADA
- U3 pad 25: unconnected-(U3-PC5-Pad25) -> ENC_PADB
- U3 pad 26: unconnected-(U3-PB0-Pad26) -> ROW0
- U3 pad 27: unconnected-(U3-PB1-Pad27) -> ROW1
- U3 pad 41: unconnected-(U3-PA8-Pad41) -> COL4
- U3 pad 46: SWDIO -> /SWDIO
- U3 pad 49: SWCLK -> /SWCLK
- U3 pad 55: unconnected-(U3-PB3-Pad55) -> ROW2
- U3 pad 56: unconnected-(U3-PB4-Pad56) -> ROW3
Other:
- board size 156.1 x 117.1 mm -> 138.1 x 128.6 mm

Commit message: Schematic Rev 1 done
Parts:
- added C17: 10u, Capacitor_SMD:C_0805_2012Metric, F.Cu at (146.1, 189.2)
- added C18: 22n, Capacitor_SMD:C_0805_2012Metric, F.Cu at (140.7, 184.2)
- added C19: 22n, Capacitor_SMD:C_0805_2012Metric, F.Cu at (145.1, 184.2)
- added J3: Conn_01x04_Pin, Connector_PinHeader_2.54mm:PinHeader_1x04_P2.54mm_Vertical, F.Cu at (91.4, 161.3)
- added R5: 1k, Resistor_SMD:R_0805_2012Metric, F.Cu at (140.1, 190.1)
- added R6: 1k, Resistor_SMD:R_0805_2012Metric, F.Cu at (140.1, 193.0)
- added R7: 10k, Resistor_SMD:R_0402_1005Metric, F.Cu at (130.1, 165.1)
- C10: footprint Capacitor_SMD:C_1206_3216Metric -> Capacitor_SMD:C_0805_2012Metric
- D10, D12, D13, D14, D15, D17, D18, D2, D20, D22, D23, D25, D3, D5, D7, D8: footprint Diode_SMD:D_SOD-123F -> Diode_SMD:D_MELF
- SW1: value SW_SPDT -> SW_BOOT
- U1: footprint Acheron_Components:USON-10_2.5x1.0mm_P0.5mm -> Package_SON:USON-10_2.5x1.0mm_P0.5mm
- moved J2 13.8 mm to (100.3, 158.8)
Connections:
- net ENC_PADA renamed BOURNS_PADA
- net ENC_PADB renamed BOURNS_PADB
- J1 pad A6: DA+ -> USB+
- J1 pad A7: DA- -> USB-
- J1 pad B6: DA+ -> USB+
- J1 pad B7: DA+ -> USB-
- SW3 pad 3: +3.3V -> VCC
- U1 pad 1: DA+ -> USB+
- U1 pad 10: DA+ -> USB+
- U1 pad 2: DA- -> USB-
- U1 pad 4: DA+ -> USB+
- U1 pad 5: DA+ -> USB+
- U1 pad 6: DA+ -> USB+
- U1 pad 7: DA+ -> USB+
- U1 pad 9: DA- -> USB-
- U3 pad 28: unconnected-(U3-PB2-Pad28) -> Net-(U3-PB2)
- U3 pad 42: unconnected-(U3-PA9-Pad42) -> Net-(J3-Pin_2)
- U3 pad 43: unconnected-(U3-PA10-Pad43) -> Net-(J3-Pin_3)
- U3 pad 44: DA- -> USB-
- U3 pad 45: DA+ -> USB+
Other:
- board text added: "BOOT→"

Commit message: Finalizing PCB
Parts:
- C12, C15, C16: footprint Capacitor_SMD:C_0805_2012Metric -> Capacitor_SMD:C_0402_1005Metric
- D1: renamed from D2; footprint Diode_SMD:D_MELF -> Diode_SMD:D_SOD-123F
- D10: renamed from D13; footprint Diode_SMD:D_MELF -> Diode_SMD:D_SOD-123F
- D11: renamed from D14; footprint Diode_SMD:D_MELF -> Diode_SMD:D_SOD-123F
- D12: renamed from D15; footprint Diode_SMD:D_MELF -> Diode_SMD:D_SOD-123F
- D13: renamed from D17; footprint Diode_SMD:D_MELF -> Diode_SMD:D_SOD-123F
- D14: renamed from D18; footprint Diode_SMD:D_MELF -> Diode_SMD:D_SOD-123F
- D16: renamed from D20; footprint Diode_SMD:D_MELF -> Diode_SMD:D_SOD-123F
- D17: renamed from D22; footprint Diode_SMD:D_MELF -> Diode_SMD:D_SOD-123F
- D18: renamed from D23; footprint Diode_SMD:D_MELF -> Diode_SMD:D_SOD-123F
- D2: renamed from D3; footprint Diode_SMD:D_MELF -> Diode_SMD:D_SOD-123F
- D20: renamed from D25; footprint Diode_SMD:D_MELF -> Diode_SMD:D_SOD-123F
- D4: renamed from D5; footprint Diode_SMD:D_MELF -> Diode_SMD:D_SOD-123F
- D5: renamed from D7; footprint Diode_SMD:D_MELF -> Diode_SMD:D_SOD-123F
- D6: renamed from D8; footprint Diode_SMD:D_MELF -> Diode_SMD:D_SOD-123F
- D8: renamed from D10; footprint Diode_SMD:D_MELF -> Diode_SMD:D_SOD-123F
- D9: renamed from D12; footprint Diode_SMD:D_MELF -> Diode_SMD:D_SOD-123F
- J2, J3: moved to B.Cu
- moved DP1 148.0 mm to (222.9, 103.9), turned to 90 degrees
- moved F1 135.1 mm to (219.2, 100.8), turned to -90 degrees
- moved R1 127.1 mm to (214.8, 109.2), turned to -90 degrees
- moved R2 123.8 mm to (208.6, 109.1), turned to -90 degrees
- moved L1 123.3 mm to (218.2, 106.7), turned to 90 degrees
- moved U1 116.9 mm to (211.6, 106.4), turned to 90 degrees
- moved U2 116.6 mm to (209.7, 142.4)
- moved R3 113.9 mm to (215.1, 143.6), turned to 180 degrees
- moved C1 113.7 mm to (218.8, 122.4), turned to -90 degrees
- moved U4 111.3 mm to (212.1, 123.2), turned to 180 degrees
- moved J1 108.3 mm to (211.6, 105.0), turned to 180 degrees
- moved C4 103.7 mm to (215.1, 141.5)
- moved C2 102.2 mm to (205.6, 124.7), turned to -90 degrees
- moved J3 97.0 mm to (188.1, 168.9), turned to 180 degrees
- moved C3 93.0 mm to (204.8, 141.5)
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- renumbered D1 to DP1
Connections:
- J1 pad B4: unconnected-(J1-VBUS-PadB4) -> VBUS
- U1 pad 5: USB+ -> USB-
- U1 pad 6: USB+ -> USB-
- U3 pad 24: BOURNS_PADA -> unconnected-(U3-PC4-Pad24)
- U3 pad 25: BOURNS_PADB -> unconnected-(U3-PC5-Pad25)
- U3 pad 26: ROW0 -> unconnected-(U3-PB0-Pad26)
- U3 pad 27: ROW1 -> unconnected-(U3-PB1-Pad27)
- U3 pad 33: unconnected-(U3-PB12-Pad33) -> ROW3
- U3 pad 41: COL4 -> unconnected-(U3-PA8-Pad41)
- U3 pad 51: unconnected-(U3-PC10-Pad51) -> ROW2
- U3 pad 52: unconnected-(U3-PC11-Pad52) -> ROW1
- U3 pad 53: unconnected-(U3-PC12-Pad53) -> ROW0
- U3 pad 54: unconnected-(U3-PD2-Pad54) -> COL4
- U3 pad 55: ROW2 -> unconnected-(U3-PB3-Pad55)
- U3 pad 56: ROW3 -> unconnected-(U3-PB4-Pad56)
- U3 pad 8: unconnected-(U3-PC0-Pad8) -> BOURNS_PADA
- U3 pad 9: unconnected-(U3-PC1-Pad9) -> BOURNS_PADB
Routing:
- net VCC: track 0.00 -> 367.9 mm, vias 0 -> 5
- net COL1: track 0.00 -> 299.0 mm, vias 0 -> 4
- net COL0: track 0.00 -> 298.3 mm
- net COL2: track 0.00 -> 263.9 mm, vias 0 -> 4
- net +3.3V: track 0.00 -> 255.1 mm
- net COL4: track 0.00 -> 169.1 mm, vias 0 -> 2
- net ROW3: track 0.00 -> 160.6 mm, vias 0 -> 2
- net USB-: track 0.00 -> 159.5 mm
- net USB+: track 0.00 -> 158.8 mm
- net COL3: track 0.00 -> 156.4 mm, vias 0 -> 2
- net ROW0: track 0.00 -> 154.1 mm, vias 0 -> 2
- net RGB_3V3: track 0.00 -> 127.0 mm, vias 0 -> 2
- net ROW1: track 0.00 -> 122.8 mm, vias 0 -> 10
- net BOURNS_PADA: track 0.00 -> 115.7 mm, vias 0 -> 7
- net Net-(DL4-DOUT): track 0.00 -> 109.7 mm, vias 0 -> 8
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- added copper zone on F.Cu, net +3.3V
- added copper zone on B.Cu, net GND
- added copper zone on F.Cu, net GNDPWR
- added copper zone on F.Cu, net VCC
Other:
- board text added: "vmacpad 0.1 cr M.Elfner github max3-2"

Commit message: Final tweaks
Parts:
- moved C15 4.96 mm to (96.0, 183.0), turned to 90 degrees
- moved C16 2.54 mm to (97.8, 189.6), turned to -90 degrees
- moved Y1 1.70 mm to (96.9, 186.3)
Routing:
- net GND: track 78.3 -> 65.2 mm, vias 24 -> 26
- net OSC_IN: track 12.6 -> 11.2 mm
- net OSC_OUT: track 10.0 -> 9.30 mm
- added copper zone on F.Cu, net GND
Other:
- board size 138.1 x 128.6 mm -> 134.7 x 126.1 mm
